File: led_breakout/led_breakout.kicad_pcb (KiCad board)
At the start: 2 copper layers, 30.5 x 30.5 mm, 19 parts, among them J1 S-, J2 P, J3 P, J4 S+

Commit message: Fix PCB errors after first assembly
Parts:
- D1: footprint LED_SMD:LED_1210_3225Metric_Pad1.42x2.65mm_HandSolder -> LED_SMD:LED_Cree-XH
- R1: value R -> 100
- R2, R3: value R -> np
- R4: value R -> 0
Connections:
- JP1 pad 1: /VCC -> Net-(D1-Pad2)
- JP5 pad 2: /VCC -> Net-(D1-Pad2)
- JP6 pad 1: /VCC -> Net-(JP6-Pad1)
- R2 pad 2: /VCC -> Net-(JP6-Pad1)
- R4 pad 2: /VCC -> Net-(JP6-Pad1)
Routing:
- net Net-(JP6-Pad1): track 0.00 -> 11.3 mm
- net Net-(D1-Pad2): track 16.1 -> 25.2 mm
- net Net-(J3-Pad1): track 0.00 -> 7.53 mm
- added copper zone on F.Cu, net Net-(D1-Pad2)
- removed copper zone on F.Cu, net /VCC
